Commit message: update: multi-jackal fix

File: src/multi_jackal/multi_jackal_description/urdf/accessories/bridge_plate.urdf.xacro (robot description, xacro)
@@ -2,10 +2,10 @@
 <robot xmlns:xacro="http://www.ros.org/wiki/xacro">
   <xacro:macro name="bridge_plate" params="mount height">
-    <joint name="${mount}_mount_to_${mount}_bridge" type="fixed">
-      <parent link="${mount}_mount"/>
-      <child link="${mount}_bridge"/>
+    <joint name="$(arg namespace)/${mount}_mount_to_${mount}_bridge" type="fixed">
+      <parent link="$(arg namespace)/${mount}_mount"/>
+      <child link="$(arg namespace)/${mount}_bridge"/>
       <origin xyz="0.0 0.0 ${height}" rpy="0 0 0"/>
     </joint>
-    <link name="${mount}_bridge">
+    <link name="$(arg namespace)/${mount}_bridge">
       <visual>
         <origin xyz="0 0 0" rpy="1.5707 0.0 1.5707" />
@@ -16,5 +16,5 @@
       </visual>
     </link>
-    <standoff_box mount="${mount}" height="${height}" />
+    <standoff_box mount="$(arg namespace)/${mount}" height="${height}" />
   </xacro:macro>
 </robot>

File: src/multi_jackal/multi_jackal_description/urdf/accessories/standoffs.urdf.xacro (robot description, xacro)
@@ -19,15 +19,15 @@
   </xacro:macro>
   <!-- Generate a set of four standoffs from a payload mount point. -->
-  <xacro:macro name="standoff_box" params="mount height">
-    <standoff name="${mount}_standoff0" length="${height}" parent="${mount}_mount">
+  <xacro:macro name="$(arg namespace)/standoff_box" params="mount height">
+    <standoff name="$(arg namespace)/${mount}_standoff0" length="${height}" parent="$(arg namespace)/${mount}_mount">
       <origin xyz="0.060 0.060 0" rpy="0 0 0"/>
     </standoff>
-    <standoff name="${mount}_standoff1" length="${height}" parent="${mount}_mount">
+    <standoff name="$(arg namespace)/${mount}_standoff1" length="${height}" parent="$(arg namespace)/${mount}_mount">
       <origin xyz="0.060 -0.060 0" rpy="0 0 0"/>
     </standoff>
-    <standoff name="${mount}_standoff2" length="${height}" parent="${mount}_mount">
+    <standoff name="$(arg namespace)/${mount}_standoff2" length="${height}" parent="$(arg namespace)/${mount}_mount">
       <origin xyz="-0.060 0.060 0" rpy="0 0 0"/>
     </standoff>
-    <standoff name="${mount}_standoff3" length="${height}" parent="${mount}_mount">
+    <standoff name="$(arg namespace)/${mount}_standoff3" length="${height}" parent="$(arg namespace)/${mount}_mount">
       <origin xyz="-0.060 -0.060 0" rpy="0 0 0"/>
     </standoff>

File: src/multi_jackal/multi_jackal_description/urdf/base_accessories.urdf.xacro (robot description, xacro)
@@ -5,67 +5,3 @@
   <!-- This optional plate mounts both the upgraded GPS and the Velodyne 3D LIDAR. -->
   <xacro:include filename="accessories/bridge_plate.urdf.xacro" />
-  <!-- If enabled, generate the LASER payload (by default, a SICK LMS111). -->
-  <xacro:include filename="accessories/sick_lms1xx_mount.urdf.xacro" />
-  <xacro:if value="$(optenv JACKAL_LASER 0)">
-    <sick_lms1xx_mount prefix="$(optenv JACKAL_LASER_MOUNT front)"
-                       topic="$(optenv JACKAL_LASER_TOPIC front/scan)"/>
-    <joint name="$(optenv JACKAL_LASER_MOUNT front)_laser_mount_joint" type="fixed">
-      <origin xyz="$(optenv JACKAL_LASER_OFFSET 0 0 0)"
-              rpy="$(optenv JACKAL_LASER_RPY 0 0 0)" />
-      <parent link="$(optenv JACKAL_LASER_MOUNT front)_mount" />
-      <child link="$(optenv JACKAL_LASER_MOUNT front)_laser_mount" />
-    </joint>
-  </xacro:if>
-  <!-- If enabled, generate the upgraded Navsat payload (a Novatel Smart6). -->
-  <xacro:include filename="accessories/novatel_smart6.urdf.xacro" />
-  <xacro:if value="$(optenv JACKAL_NAVSAT 0)">
-    <bridge_plate mount="$(optenv JACKAL_NAVSAT_MOUNT rear)"
-                  height="$(optenv JACKAL_NAVSAT_HEIGHT 0.1)" />
-    <novatel_smart6 prefix="$(optenv JACKAL_NAVSAT_MOUNT rear)"/>
-    <joint name="$(optenv JACKAL_NAVSAT_MOUNT rear)_navsat_joint" type="fixed">
-      <origin xyz="0 0 0" rpy="0 0 0" />
-      <parent link="$(optenv JACKAL_NAVSAT_MOUNT rear)_bridge" />
-      <child link="$(optenv JACKAL_NAVSAT_MOUNT rear)_navsat" />
-    </joint>
-  </xacro:if>
-  <!-- If enabled, generate the flea3 camera payload with a tilt of 30 degrees. -->
-  <xacro:include filename="accessories/camera_mount.urdf.xacro" />
-  <xacro:include filename="$(find pointgrey_camera_description)/urdf/pointgrey_flea3.urdf.xacro" />
-  <xacro:if value="$(optenv JACKAL_FLEA3 0)">
-    <camera_mount prefix="$(optenv JACKAL_FLEA_MOUNT front)"
-                       tilt="$(optenv JACKAL_FLEA_TILT 0)"/>
-    <joint name="$(optenv JACKAL_FLEA3_MOUNT front)_camera_mount_joint" type="fixed">
-      <origin xyz="$(optenv JACKAL_FLEA3_OFFSET 0 0 0)"
-              rpy="$(optenv JACKAL_FLEA3_RPY 0 0 0)" />
-      <parent link="$(optenv JACKAL_FLEA_MOUNT front)_mount" />
-      <child link="$(optenv JACKAL_FLEA_MOUNT front)_camera_mount" />
-    </joint>
-    <pointgrey_flea3 frame="$(optenv JACKAL_FLEA3_MOUNT front)_camera" name="$(optenv JACKAL_FLEA_NAME front)"
-      camera_x="0.0754" camera_y="0.029" camera_z="0.035"
-      camera_mass="0.085" hfov="1.0471975512" fps="60" width="640" height="512"/>
-    <joint name="$(optenv JACKAL_FLEA3_MOUNT front)_camera_bracket_joint" type="fixed">
-      <origin xyz="0.020 0 0.0245" rpy="0 0 0" />
-      <parent link="$(optenv JACKAL_FLEA3_MOUNT front)_camera_beam" />
-      <child link="$(optenv JACKAL_FLEA3_MOUNT front)_camera" />
-    </joint>
-  </xacro:if>
-  <!-- If enabled, generate the bumblebee2 camera payload with a tilt of 0 degrees. -->
-  <xacro:include filename="accessories/camera_mount.urdf.xacro" />
-  <xacro:include filename="$(find pointgrey_camera_description)/urdf/pointgrey_bumblebee2.urdf.xacro" />
-  <xacro:if value="$(optenv JACKAL_BB2 0)">
-    <camera_mount prefix="$(optenv JACKAL_BB2_MOUNT front)"
-                        tilt="$(optenv JACKAL_BB2_TILT 0)"/>
-    <joint name="$(optenv JACKAL_BB2_MOUNT front)_camera_mount_joint" type="fixed">
-      <origin xyz="$(optenv JACKAL_BB2_OFFSET 0 0 0)"
-              rpy="$(optenv JACKAL_BB2_RPY 0 0 0)" />
-      <parent link="$(optenv JACKAL_BB2_MOUNT front)_mount" />
-      <child link="$(optenv JACKAL_BB2_MOUNT front)_camera_mount" />
-    </joint>
-    <BB2-08S2C-38 frame="$(optenv JACKAL_BB2_MOUNT front)_camera" name="$(optenv JACKAL_BB2_NAME front)" />
-    <joint name="$(optenv JACKAL_BB2_MOUNT front)_camera_bracket_joint" type="fixed">
-      <origin xyz="0.007 0 0.02450" rpy="0 0 0" />
-      <parent link="$(optenv JACKAL_BB2_MOUNT front)_camera_beam" />
-      <child link="$(optenv JACKAL_BB2_MOUNT front)_camera" />
-    </joint>
-  </xacro:if>
 </robot>

File: src/multi_jackal/multi_jackal_description/urdf/custom_accessories.urdf.xacro (robot description, xacro)
@@ -5,20 +5,7 @@
        The accessory can then be enabled by setting the 'config' argument in the
        launch files. -->
-  <!-- Box with AprilTag markers on each face. -->
-  <xacro:if value="$(optenv JACKAL_APRILTAG 0)">
-    <xacro:include filename="accessories/apriltag_box.urdf.xacro" />
-  </xacro:if>
-  <!-- Box with ARTrackAlvar markers on each face. -->
-  <xacro:if value="$(optenv JACKAL_ALVARTAG 0)">
-    <xacro:include filename="accessories/alvartag_box.urdf.xacro" />
-  </xacro:if>
-  <!-- Front and rear cameras. -->
-  <xacro:if value="$(optenv JACKAL_TWOCAMS 0)">
-    <xacro:include filename="accessories/camera_mount.urdf.xacro" />
-    <xacro:include filename="accessories/twocams.urdf.xacro"/>
-  </xacro:if>
-  <!-- Box with AprilTag markers on each face, lifted up slightly. -->
-  <xacro:if value="$(optenv JACKAL_APRILTAG_POLE 0)">
-    <xacro:include filename="accessories/apriltag_box_with_pole.urdf.xacro" />
-  </xacro:if>
+    <!-- Box with AprilTag markers on each face, lifted up slightly. -->
+    <xacro:if value="$(optenv SHEFFIELD_ROBOT 0)">
+      <xacro:include filename="$(find shef04_jackal)/urdf/jackal_description.urdf.xacro" />
+    </xacro:if>
 </robot>

File: src/multi_jackal/multi_jackal_description/urdf/jackal.urdf.xacro (robot description, xacro)
@@ -49,5 +49,5 @@
     </gazebo>
     <joint name="${prefix}_wheel" type="continuous">
-      <parent link="chassis_link"/>
+      <parent link="$(arg namespace)/chassis_link"/>
       <child link="${prefix}_wheel_link" />
       <xacro:insert_block name="joint_pose" />
@@ -67,23 +67,23 @@
   </xacro:macro>
   <!-- The joints and links. -->
-  <xacro:wheel prefix="front_left">
+  <xacro:wheel prefix="$(arg namespace)/front_left">
     <origin xyz="${wheelbase/2} ${track/2} ${wheel_vertical_offset}" rpy="0 0 0" />
   </xacro:wheel>
-  <xacro:wheel prefix="front_right">
+  <xacro:wheel prefix="$(arg namespace)/front_right">
     <origin xyz="${wheelbase/2} ${-track/2} ${wheel_vertical_offset}" rpy="0 0 0" />
   </xacro:wheel>
-  <xacro:wheel prefix="rear_left">
+  <xacro:wheel prefix="$(arg namespace)/rear_left">
     <origin xyz="${-wheelbase/2} ${track/2} ${wheel_vertical_offset}" rpy="0 0 0" />
   </xacro:wheel>
-  <xacro:wheel prefix="rear_right">
+  <xacro:wheel prefix="$(arg namespace)/rear_right">
     <origin xyz="${-wheelbase/2} ${-track/2} ${wheel_vertical_offset}" rpy="0 0 0" />
   </xacro:wheel>
-  <link name="base_link"></link>
-  <joint name="base_link_joint" type="fixed">
+  <link name="$(arg namespace)/base_link"></link>
+  <joint name="$(arg namespace)/base_link_joint" type="fixed">
     <origin xyz="0 0 0" rpy="0 0 0" />
-    <parent link="base_link"/>
-    <child link="chassis_link" />
+    <parent link="$(arg namespace)/base_link"/>
+    <child link="$(arg namespace)/chassis_link" />
   </joint>
-  <link name="chassis_link">
+  <link name="$(arg namespace)/chassis_link">
     <visual>
       <origin xyz="0 0 ${footprint_vertical_offset}" rpy="${PI/2} 0 ${PI/2}"/>
@@ -110,5 +110,5 @@
       </inertial>
   </link>
-  <link name="fenders_link">
+  <link name="$(arg namespace)/fenders_link">
     <visual>
       <origin xyz="0 0 ${footprint_vertical_offset}" rpy="${PI/2} 0 ${PI/2}"/>
@@ -119,7 +119,7 @@
     </visual>
   </link>
-  <joint name="fenders_joint" type="fixed">
-    <parent link="chassis_link" />
-    <child link="fenders_link" />
+  <joint name="$(arg namespace)/fenders_joint" type="fixed">
+    <parent link="$(arg namespace)/chassis_link" />
+    <child link="$(arg namespace)/fenders_link" />
   </joint>
   <!-- TODO: Make this internal_imu_link or something, and use a mixed-in xacro
@@ -127,5 +127,5 @@
        always points to the "active" IMU. When an upgrade IMU is connected, the
        internal_imu_link should remain, but imu_link should point to the upgrade one. -->
-  <link name="imu_link">
+  <link name="$(arg namespace)/imu_link">
     <inertial>
       <mass value="0.001"/>
@@ -134,10 +134,10 @@
     </inertial>
   </link>
-  <joint name="imu_joint" type="fixed">
-    <parent link="chassis_link" />
-    <child link="imu_link" />
+  <joint name="$(arg namespace)/imu_joint" type="fixed">
+    <parent link="$(arg namespace)/chassis_link" />
+    <child link="$(arg namespace)/imu_link" />
   </joint>
   <!-- TODO: Same note as applies to imu_link -->
-  <link name="navsat_link">
+  <link name="$(arg namespace)/navsat_link">
     <visual>
       <geometry>
@@ -148,25 +148,25 @@
     </visual>
   </link>
-  <joint name="navsat_joint" type="fixed">
-    <parent link="chassis_link" />
-    <child link="navsat_link" />
+  <joint name="$(arg namespace)/navsat_joint" type="fixed">
+    <parent link="$(arg namespace)/chassis_link" />
+    <child link="$(arg namespace)/navsat_link" />
     <origin xyz="-0.180 0.126 0.1815" />
   </joint>
-  <link name="mid_mount"></link>
-  <joint name="mid_mount_joint" type="fixed">
-    <parent link="chassis_link" />
-    <child link="mid_mount" />
+  <link name="$(arg namespace)/mid_mount"></link>
+  <joint name="$(arg namespace)/mid_mount_joint" type="fixed">
+    <parent link="$(arg namespace)/chassis_link" />
+    <child link="$(arg namespace)/mid_mount" />
     <origin xyz="0 0 ${chassis_height}" />
   </joint>
-  <link name="rear_mount"></link>
-  <joint name="rear_mount_joint" type="fixed">
-    <parent link="mid_mount" />
-    <child link="rear_mount" />
+  <link name="$(arg namespace)/rear_mount"></link>
+  <joint name="$(arg namespace)/rear_mount_joint" type="fixed">
+    <parent link="$(arg namespace)/mid_mount" />
+    <child link="$(arg namespace)/rear_mount" />
     <origin xyz="${-mount_spacing} 0 0" />
   </joint>
-  <link name="front_mount"></link>
-  <joint name="front_mount_joint" type="fixed">
-    <parent link="mid_mount" />
-    <child link="front_mount" />
+  <link name="$(arg namespace)/front_mount"></link>
+  <joint name="$(arg namespace)/front_mount_joint" type="fixed">
+    <parent link="$(arg namespace)/mid_mount" />
+    <child link="$(arg namespace)/front_mount" />
     <origin xyz="${mount_spacing} 0 0" />
   </joint>
