Commit message: update: pallet limits

File: src/jackal_workspace/urdf/pallet.urdf.xacro (robot description, xacro)
@@ -46,5 +46,5 @@
         <axis xyz="0.0 0.0 1.0" />
         <dynamics damping="1.0" friction="5.0" />
-        <limit lower="-1.57" upper="1.57" effort="100.0" velocity="10.0" />
+        <limit lower="-3.1" upper="3.1" effort="100.0" velocity="10.0" />
     </joint>
     <link name="straigth_bar_one">
@@ -82,5 +82,5 @@
         <axis xyz="0.0 0.0 1.0" />
         <dynamics damping="1.0" friction="5.0" />
-        <limit lower="-1.57" upper="1.57" effort="100.0" velocity="10.0" />
+        <limit lower="-3.1" upper="3.1" effort="100.0" velocity="10.0" />
     </joint>
     <link name="connector_robot_two">
@@ -100,5 +100,5 @@
         <axis xyz="0.0 0.0 1.0" />
         <dynamics damping="1.0" friction="5.0" />
-        <limit lower="-1.57" upper="1.57" effort="100.0" velocity="10.0" />
+        <limit lower="-3.1" upper="3.1" effort="100.0" velocity="10.0" />
     </joint>
     <link name="straigth_bar_two">
@@ -136,5 +136,5 @@
         <axis xyz="0.0 0.0 1.0" />
         <dynamics damping="1.0" friction="5.0" />
-        <limit lower="-1.57" upper="1.57" effort="100.0" velocity="10.0" />
+        <limit lower="-3.1" upper="3.1" effort="100.0" velocity="10.0" />
     </joint>
 </robot>

File: src/velodyne_simulator/velodyne_description/urdf/VLP-16.urdf.xacro (robot description, xacro)
@@ -2,5 +2,5 @@
 <robot xmlns:xacro="http://www.ros.org/wiki/xacro" name="VLP-16">
   <xacro:property name="M_PI" value="3.1415926535897931" />
-  <xacro:macro name="VLP-16" params="*origin parent:=base_link name:=velodyne topic:=/velodyne_points organize_cloud:=false hz:=10 lasers:=16 samples:=1875 collision_range:=0.3 min_range:=0.9 max_range:=130.0 noise:=0.008 min_angle:=-${M_PI} max_angle:=${M_PI} gpu:=false">
+  <xacro:macro name="VLP-16" params="*origin parent:=base_link name:=velodyne topic:=/velodyne_points organize_cloud:=false hz:=10 lasers:=16 samples:=1875 collision_range:=0.3 min_range:=0.9 max_range:=130.0 noise:=0.008 min_angle:=-${M_PI} max_angle:=${M_PI} gpu:=true">
     <joint name="${name}_base_mount_joint" type="fixed">
       <xacro:insert_block name="origin" />

Commit message: update: pallet pose

File: src/jackal_workspace/urdf/pallet.urdf.xacro (robot description, xacro)
@@ -11,8 +11,18 @@
         <color rgba="1.0 1.0 1.0 1.0" />
     </material>
+    <gazebo>
+        <plugin name="nexus_custom_force_based_move" filename="libfeedback.so">
+          <commandTopic>cmd_vel</commandTopic>
+          <poseTopic>goal</poseTopic>
+          <odometryTopic>pallet_pose</odometryTopic>
+          <odometryFrame>map</odometryFrame>
+          <odometryRate>30.0</odometryRate>
+          <robotBaseFrame>pallet</robotBaseFrame>
+        </plugin>
+     </gazebo>
     <link name="pallet">
         <inertial>
             <origin xyz="0.0 0.0 0.0" rpy="0.0 0.0 0.0" />
-            <mass value="10.0" />
+            <mass value="5.0" />
             <inertia ixx="2.43" ixy="0.0" ixz="0.0" iyy="1.10" iyz="0.0" izz="3.47" />
         </inertial>
@@ -45,6 +55,6 @@
         <child link="connector_robot_one" />
         <axis xyz="0.0 0.0 1.0" />
-        <dynamics damping="1.0" friction="5.0" />
-        <limit lower="-3.1" upper="3.1" effort="100.0" velocity="10.0" />
+        <dynamics damping="0.5" friction="1.0" />
+        <limit lower="-3.1" upper="3.1" effort="10.0" velocity="10.0" />
     </joint>
     <link name="straigth_bar_one">
@@ -63,6 +73,6 @@
         <child link="straigth_bar_one" />
         <axis xyz="1.0 0.0 0.0" />
-        <dynamics damping="10.0" friction="100.0" />
-        <limit lower="-0.5" upper="0.7" effort="1000.0" velocity="10.0" />
+        <dynamics damping="0.5" friction="1.0" />
+        <limit lower="-0.5" upper="0.7" effort="10.0" velocity="10.0" />
     </joint>
     <link name="connector_bar_one">
@@ -81,6 +91,6 @@
         <child link="connector_bar_one" />
         <axis xyz="0.0 0.0 1.0" />
-        <dynamics damping="1.0" friction="5.0" />
-        <limit lower="-3.1" upper="3.1" effort="100.0" velocity="10.0" />
+        <dynamics damping="0.5" friction="1.0" />
+        <limit lower="-3.1" upper="3.1" effort="10.0" velocity="10.0" />
     </joint>
     <link name="connector_robot_two">
@@ -99,6 +109,6 @@
         <child link="connector_robot_two" />
         <axis xyz="0.0 0.0 1.0" />
-        <dynamics damping="1.0" friction="5.0" />
-        <limit lower="-3.1" upper="3.1" effort="100.0" velocity="10.0" />
+        <dynamics damping="0.5" friction="1.0" />
+        <limit lower="-3.1" upper="3.1" effort="10.0" velocity="10.0" />
     </joint>
     <link name="straigth_bar_two">
@@ -117,6 +127,6 @@
         <child link="straigth_bar_two" />
         <axis xyz="1.0 0.0 0.0" />
-        <dynamics damping="10.0" friction="100.0" />
-        <limit lower="-0.5" upper="0.7" effort="1000.0" velocity="10.0" />
+        <dynamics damping="0.5" friction="1.0" />
+        <limit lower="-0.5" upper="0.7" effort="10.0" velocity="10.0" />
     </joint>
     <link name="connector_bar_two">
@@ -135,6 +145,6 @@
         <child link="connector_bar_two" />
         <axis xyz="0.0 0.0 1.0" />
-        <dynamics damping="1.0" friction="5.0" />
-        <limit lower="-3.1" upper="3.1" effort="100.0" velocity="10.0" />
+        <dynamics damping="0.5" friction="1.0" />
+        <limit lower="-3.1" upper="3.1" effort="10.0" velocity="10.0" />
     </joint>
 </robot>

File: src/multi_jackal/multi_jackal_description/urdf/jackal.urdf.xacro (robot description, xacro)
@@ -102,5 +102,5 @@
       <!-- Center of mass -->
       <origin xyz="0.012  0.002 0.067" rpy="0 0 0"/>
-      <mass value="16.523"/>
+      <mass value="26.523"/>
       <!-- Moments of inertia: ( chassis without wheels ) -->
       <inertia

Commit message: update: local and global planner

File: src/jackal_workspace/urdf/pallet.urdf.xacro (robot description, xacro)
@@ -59,9 +59,9 @@
     </joint>
     <link name="straigth_bar_one">
-        <xacro:inertial_cuboid mass="1.0" x_length="1.5" y_length="0.01" z_length="0.01" />
+        <xacro:inertial_cuboid mass="1.0" x_length="0.6" y_length="0.01" z_length="0.01" />
         <visual>
-            <origin xyz="0.0 0.0 0.0" rpy="0.0 0.0 0.0" />
+            <origin xyz="0.3 0.0 0.0" rpy="0.0 0.0 0.0" />
             <geometry>
-                <box size="1.5 0.01 0.01" />
+                <box size="0.6 0.01 0.01" />
             </geometry>
             <material name="dark_grey" />
@@ -74,5 +74,5 @@
         <axis xyz="1.0 0.0 0.0" />
         <dynamics damping="0.5" friction="1.0" />
-        <limit lower="-0.5" upper="0.7" effort="10.0" velocity="10.0" />
+        <limit lower="-0.6" upper="0.0" effort="10.0" velocity="10.0" />
     </joint>
     <link name="connector_bar_one">
@@ -87,5 +87,5 @@
     </link>
     <joint name="connector_bar_one_joint" type="revolute">
-        <origin xyz="0.75 0.0 0.0" rpy="0.0 0.0 0.0" />
+        <origin xyz="0.6 0.0 0.0" rpy="0.0 0.0 0.0" />
         <parent link="straigth_bar_one" />
         <child link="connector_bar_one" />
@@ -113,9 +113,9 @@
     </joint>
     <link name="straigth_bar_two">
-        <xacro:inertial_cuboid mass="1.0" x_length="1.5" y_length="0.01" z_length="0.01" />
+        <xacro:inertial_cuboid mass="1.0" x_length="0.6" y_length="0.01" z_length="0.01" />
         <visual>
-            <origin xyz="0.0 0.0 0.0" rpy="0.0 0.0 0.0" />
+            <origin xyz="0.3 0.0 0.0" rpy="0.0 0.0 0.0" />
             <geometry>
-                <box size="1.5 0.01 0.01" />
+                <box size="0.6 0.01 0.01" />
             </geometry>
             <material name="dark_grey" />
@@ -128,5 +128,5 @@
         <axis xyz="1.0 0.0 0.0" />
         <dynamics damping="0.5" friction="1.0" />
-        <limit lower="-0.5" upper="0.7" effort="10.0" velocity="10.0" />
+        <limit lower="-0.6" upper="0.0" effort="10.0" velocity="10.0" />
     </joint>
     <link name="connector_bar_two">
@@ -141,5 +141,5 @@
     </link>
     <joint name="connector_bar_two_joint" type="revolute">
-        <origin xyz="0.75 0.0 0.0" rpy="0.0 0.0 0.0" />
+        <origin xyz="0.6 0.0 0.0" rpy="0.0 0.0 0.0" />
         <parent link="straigth_bar_two" />
         <child link="connector_bar_two" />
