Commit message: update: mapt controller update

File: src/jackal_workspace/urdf/pallet1bar.urdf.xacro (robot description, xacro)
@@ -55,5 +55,5 @@
         <child link="connector_robot_one" />
         <axis xyz="0.0 0.0 1.0" />
-        <dynamics damping="0.5" friction="1.0" />
+        <dynamics damping="0.1" friction="0.5" />
         <limit lower="-3.1" upper="3.1" effort="10.0" velocity="10.0" />
     </joint>
@@ -73,5 +73,5 @@
         <child link="straigth_bar_one" />
         <axis xyz="1.0 0.0 0.0" />
-        <dynamics damping="0.5" friction="1.0" />
+        <dynamics damping="0.1" friction="0.5" />
         <limit lower="-0.6" upper="0.0" effort="10.0" velocity="10.0" />
     </joint>
@@ -91,5 +91,5 @@
         <child link="connector_bar_one" />
         <axis xyz="0.0 0.0 1.0" />
-        <dynamics damping="0.5" friction="1.0" />
+        <dynamics damping="0.1" friction="0.5" />
         <limit lower="-3.1" upper="3.1" effort="10.0" velocity="10.0" />
     </joint>

File: src/jackal_workspace/urdf/pallet2bar.urdf.xacro (robot description, xacro)
@@ -40,4 +40,25 @@
         </collision>
     </link>
+    <link name="box">
+        <inertial>
+            <origin xyz="0.0 0.0 0.5" rpy="0.0 0.0 0.0" />
+            <mass value="5.0" />
+            <inertia ixx="2.43" ixy="0.0" ixz="0.0" iyy="1.10" iyz="0.0" izz="3.47" />
+        </inertial>
+        <visual>
+            <origin xyz="0.0 0.0 0.2" rpy="0.0 0.0 0.0" />
+            <geometry>
+                <box size="0.5 1.0 0.4"/>
+            </geometry>
+        </visual>
+    </link>
+    <joint name="box_pallet" type="fixed">
+        <origin xyz="0.0 0.0 0.1" rpy="0.0 0.0 0.0" />
+        <parent link="pallet" />
+        <child link="box" />
+        <axis xyz="0.0 0.0 1.0" />
+        <dynamics damping="0.1" friction="0.5" />
+        <limit lower="-3.1" upper="3.1" effort="10.0" velocity="10.0" />
+    </joint>
     <link name="connector_robot_one">
         <xacro:inertial_cuboid mass="1.0" x_length="0.05" y_length="0.05" z_length="0.05" />
@@ -55,5 +76,5 @@
         <child link="connector_robot_one" />
         <axis xyz="0.0 0.0 1.0" />
-        <dynamics damping="0.5" friction="1.0" />
+        <dynamics damping="0.1" friction="0.5" />
         <limit lower="-3.1" upper="3.1" effort="10.0" velocity="10.0" />
     </joint>
@@ -73,5 +94,5 @@
         <child link="straigth_bar_one" />
         <axis xyz="1.0 0.0 0.0" />
-        <dynamics damping="0.5" friction="1.0" />
+        <dynamics damping="0.1" friction="0.5" />
         <limit lower="-0.6" upper="0.0" effort="10.0" velocity="10.0" />
     </joint>
@@ -91,5 +112,5 @@
         <child link="connector_bar_one" />
         <axis xyz="0.0 0.0 1.0" />
-        <dynamics damping="0.5" friction="1.0" />
+        <dynamics damping="0.1" friction="0.5" />
         <limit lower="-3.1" upper="3.1" effort="10.0" velocity="10.0" />
     </joint>
@@ -109,5 +130,5 @@
         <child link="connector_robot_two" />
         <axis xyz="0.0 0.0 1.0" />
-        <dynamics damping="0.5" friction="1.0" />
+        <dynamics damping="0.1" friction="0.5" />
         <limit lower="-3.1" upper="3.1" effort="10.0" velocity="10.0" />
     </joint>
@@ -127,5 +148,5 @@
         <child link="straigth_bar_two" />
         <axis xyz="1.0 0.0 0.0" />
-        <dynamics damping="0.5" friction="1.0" />
+        <dynamics damping="0.1" friction="0.5" />
         <limit lower="-0.6" upper="0.0" effort="10.0" velocity="10.0" />
     </joint>
@@ -145,5 +166,5 @@
         <child link="connector_bar_two" />
         <axis xyz="0.0 0.0 1.0" />
-        <dynamics damping="0.5" friction="1.0" />
+        <dynamics damping="0.1" friction="0.5" />
         <limit lower="-3.1" upper="3.1" effort="10.0" velocity="10.0" />
     </joint>

File: src/jackal_workspace/urdf/pallet3bar.urdf.xacro (robot description, xacro)
@@ -40,4 +40,25 @@
         </collision>
     </link>
+    <link name="box">
+        <inertial>
+            <origin xyz="0.0 0.0 0.5" rpy="0.0 0.0 0.0" />
+            <mass value="5.0" />
+            <inertia ixx="2.43" ixy="0.0" ixz="0.0" iyy="1.10" iyz="0.0" izz="3.47" />
+        </inertial>
+        <visual>
+            <origin xyz="0.0 0.0 0.5" rpy="0.0 0.0 0.0" />
+            <geometry>
+                <box size="0.5 1.0 1.0"/>
+            </geometry>
+        </visual>
+    </link>
+    <joint name="box_pallet" type="fixed">
+        <origin xyz="0.0 0.0 0.1" rpy="0.0 0.0 0.0" />
+        <parent link="pallet" />
+        <child link="box" />
+        <axis xyz="0.0 0.0 1.0" />
+        <dynamics damping="0.1" friction="0.5" />
+        <limit lower="-3.1" upper="3.1" effort="10.0" velocity="10.0" />
+    </joint>
     <link name="connector_robot_one">
         <xacro:inertial_cuboid mass="1.0" x_length="0.05" y_length="0.05" z_length="0.05" />
@@ -55,5 +76,5 @@
         <child link="connector_robot_one" />
         <axis xyz="0.0 0.0 1.0" />
-        <dynamics damping="0.5" friction="1.0" />
+        <dynamics damping="0.1" friction="0.5" />
         <limit lower="-3.1" upper="3.1" effort="10.0" velocity="10.0" />
     </joint>
@@ -73,5 +94,5 @@
         <child link="straigth_bar_one" />
         <axis xyz="1.0 0.0 0.0" />
-        <dynamics damping="0.5" friction="1.0" />
+        <dynamics damping="0.1" friction="0.5" />
         <limit lower="-0.6" upper="0.0" effort="10.0" velocity="10.0" />
     </joint>
@@ -91,5 +112,5 @@
         <child link="connector_bar_one" />
         <axis xyz="0.0 0.0 1.0" />
-        <dynamics damping="0.5" friction="1.0" />
+        <dynamics damping="0.1" friction="0.5" />
         <limit lower="-3.1" upper="3.1" effort="10.0" velocity="10.0" />
     </joint>
@@ -109,5 +130,5 @@
         <child link="connector_robot_two" />
         <axis xyz="0.0 0.0 1.0" />
-        <dynamics damping="0.5" friction="1.0" />
+        <dynamics damping="0.1" friction="0.5" />
         <limit lower="-3.1" upper="3.1" effort="10.0" velocity="10.0" />
     </joint>
@@ -127,5 +148,5 @@
         <child link="straigth_bar_two" />
         <axis xyz="1.0 0.0 0.0" />
-        <dynamics damping="0.5" friction="1.0" />
+        <dynamics damping="0.1" friction="0.5" />
         <limit lower="-0.6" upper="0.0" effort="10.0" velocity="10.0" />
     </joint>
@@ -145,5 +166,5 @@
         <child link="connector_bar_two" />
         <axis xyz="0.0 0.0 1.0" />
-        <dynamics damping="0.5" friction="1.0" />
+        <dynamics damping="0.1" friction="0.5" />
         <limit lower="-3.1" upper="3.1" effort="10.0" velocity="10.0" />
     </joint>
@@ -164,5 +185,5 @@
         <child link="connector_robot_three" />
         <axis xyz="0.0 0.0 1.0" />
-        <dynamics damping="0.5" friction="1.0" />
+        <dynamics damping="0.1" friction="0.5" />
         <limit lower="-3.1" upper="3.1" effort="10.0" velocity="10.0" />
     </joint>
@@ -182,5 +203,5 @@
         <child link="straigth_bar_three" />
         <axis xyz="1.0 0.0 0.0" />
-        <dynamics damping="0.5" friction="1.0" />
+        <dynamics damping="0.1" friction="0.5" />
         <limit lower="-0.6" upper="0.0" effort="10.0" velocity="10.0" />
     </joint>
@@ -200,5 +221,5 @@
         <child link="connector_bar_three" />
         <axis xyz="0.0 0.0 1.0" />
-        <dynamics damping="0.5" friction="1.0" />
+        <dynamics damping="0.1" friction="0.5" />
         <limit lower="-3.1" upper="3.1" effort="10.0" velocity="10.0" />
     </joint>

File: src/shef04_jackal/urdf/jackal_description.urdf.xacro (robot description, xacro)
@@ -50,5 +50,5 @@
     <parent link="$(arg namespace)/front_mount" />
     <child link="$(arg namespace)/laser" />
-    <origin xyz="0 0 0.08" />
+    <origin xyz="0 0 0.08" rpy="0 0 0"/>
   </joint>
   <xacro:include filename="$(find velodyne_description)/urdf/VLP-16.urdf.xacro"/>
