Commit message: update : code refactor

File: src/jackal_workspace/urdf/pallet2bar.urdf.xacro (robot description, xacro)
@@ -151,5 +151,5 @@
         <limit lower="-0.6" upper="0.0" effort="10.0" velocity="10.0" />
     </joint>
-    <link name="connector_bar_two">
+    <link name="connector_bar_three">
         <xacro:inertial_cuboid mass="1.0" x_length="0.05" y_length="0.05" z_length="0.05" />
         <visual>
@@ -161,8 +161,8 @@
         </visual>
     </link>
-    <joint name="connector_bar_two_joint" type="revolute">
+    <joint name="connector_bar_three_joint" type="revolute">
         <origin xyz="0.6 0.0 0.0" rpy="0.0 0.0 0.0" />
         <parent link="straigth_bar_two" />
-        <child link="connector_bar_two" />
+        <child link="connector_bar_three" />
         <axis xyz="0.0 0.0 1.0" />
         <dynamics damping="0.1" friction="0.5" />
